Commit message: feat: update AGV robot description and simulation for Mecanum drive capabilities

File: ros2_ws/src/avg_description/urdf/robot.xacro (robot description, xacro)
@@ -172,30 +172,35 @@
   <!-- Gazebo Plugins for gz sim (Gazebo Harmonic) -->
   <!-- ========================================== -->
-  <!-- Differential drive controller plugin -->
+  <!-- Mecanum / Omni-Directional Drive controller plugin -->
   <gazebo>
-    <plugin filename="gz-sim-diff-drive-system" name="gz::sim::systems::DiffDrive">
-      <left_joint>wheel_front_left_joint</left_joint>
-      <left_joint>wheel_rear_left_joint</left_joint>
-      <right_joint>wheel_front_right_joint</right_joint>
-      <right_joint>wheel_rear_right_joint</right_joint>
+    <plugin filename="gz-sim-mecanum-drive-system" name="gz::sim::systems::MecanumDrive">
+      <!-- Wheel joint configuration (mecanum pattern) -->
+      <front_left_joint>wheel_front_left_joint</front_left_joint>
+      <front_right_joint>wheel_front_right_joint</front_right_joint>
+      <back_left_joint>wheel_rear_left_joint</back_left_joint>
+      <back_right_joint>wheel_rear_right_joint</back_right_joint>
+      <!-- Robot physical parameters -->
       <wheel_separation>${wheel_separation}</wheel_separation>
+      <wheelbase>${wheelbase}</wheelbase>
       <wheel_radius>${wheel_radius}</wheel_radius>
-      <odom_publish_frequency>50</odom_publish_frequency>
-      <max_linear_acceleration>1.0</max_linear_acceleration>
-      <min_linear_acceleration>-1.0</min_linear_acceleration>
-      <max_angular_acceleration>2.0</max_angular_acceleration>
-      <min_angular_acceleration>-2.0</min_angular_acceleration>
-      <max_linear_velocity>0.5</max_linear_velocity>
-      <min_linear_velocity>-0.5</min_linear_velocity>
-      <max_angular_velocity>1.0</max_angular_velocity>
-      <min_angular_velocity>-1.0</min_angular_velocity>
+      <!-- Velocity limits -->
+      <max_linear_velocity>1.6</max_linear_velocity>
+      <min_linear_velocity>-1.6</min_linear_velocity>
+      <max_angular_velocity>4.5</max_angular_velocity>
+      <min_angular_velocity>-4.5</min_angular_velocity>
+      <!-- Acceleration limits -->
+      <max_linear_acceleration>1.5</max_linear_acceleration>
+      <max_angular_acceleration>3.0</max_angular_acceleration>
+      <!-- ROS 2 topics -->
       <topic>cmd_vel</topic>
       <odom_topic>odom</odom_topic>
       <tf_topic>/tf</tf_topic>
+      <!-- Frame configuration -->
       <frame_id>odom</frame_id>
       <child_frame_id>base_footprint</child_frame_id>
+      <!-- Publishing configuration -->
+      <odom_publish_frequency>50</odom_publish_frequency>
       <publish_odom>true</publish_odom>
       <publish_odom_tf>true</publish_odom_tf>
-      <publish_wheel_tf>false</publish_wheel_tf>
     </plugin>
   </gazebo>

File: ros2_ws/src/avg_description/urdf/wheel_macro.xacro (robot description, xacro)
@@ -94,15 +94,26 @@
       <child link="wheel_${prefix}"/>
       <axis xyz="0 1 0"/>
-      <dynamics damping="0.1" friction="0.1"/>
+      <dynamics damping="0.05" friction="0.05"/>
     </joint>
-    <!-- Gazebo properties for the wheel -->
+    <!-- Gazebo properties for MECANUM/OMNI wheel physics -->
     <gazebo reference="wheel_${prefix}">
       <material>Gazebo/Black</material>
-      <mu1>1.0</mu1>
-      <mu2>1.0</mu2>
-      <kp>1000000.0</kp>
-      <kd>100.0</kd>
+      <!-- Omnidirectional friction (equal in all directions for mecanum) -->
+      <mu1>1.0</mu1>   <!-- Primary friction -->
+      <mu2>1.0</mu2>   <!-- Secondary friction (equal for omni movement) -->
+      <!-- Contact physics - Optimized for mecanum -->
+      <kp>1000000.0</kp>     <!-- Contact stiffness -->
+      <kd>10.0</kd>          <!-- Contact damping -->
       <minDepth>0.001</minDepth>
-      <maxVel>1.0</maxVel>
+      <maxVel>100.0</maxVel>
+      <maxContacts>1</maxContacts>  <!-- Single contact point per wheel -->
+      <!-- Mecanum wheels need some slip in all directions -->
+      <slip1>0.1</slip1>
+      <slip2>0.1</slip2>
+      <!-- Surface properties for consistent behavior -->
+      <bounce>0.0</bounce>
+      <bounce_threshold>100000</bounce_threshold>
+      <soft_cfm>0.0</soft_cfm>
+      <soft_erp>0.2</soft_erp>
     </gazebo>
   </xacro:macro>

Commit message: feat: enhance AGV robot simulation with Mecanum drive properties and joystick control settings

File: ros2_ws/src/avg_description/urdf/robot.xacro (robot description, xacro)
@@ -135,21 +135,26 @@
     </inertial>
   </link>
-  <!-- ========================================== -->
-  <!-- Wheels (Using Wheel Macro)                 -->
-  <!-- ========================================== -->
-  <!-- Front Left Wheel -->
-  <xacro:wheel prefix="front_left" parent="base_link">
+  <!-- Gazebo properties for base_link (low friction to prevent dragging) -->
+  <gazebo reference="base_link">
+    <mu1>0.000002</mu1>
+    <mu2>0.000002</mu2>
+  </gazebo>
+  <!-- ========================================== -->
+  <!-- Wheels (Using Wheel Macro with Mecanum Friction) -->
+  <!-- ========================================== -->
+  <!-- Front Left Wheel - friction direction (1, -1, 0) -->
+  <xacro:wheel prefix="front_left" parent="base_link" friction_dir="1 -1 0">
     <origin xyz="${wheel_x_offset_front} ${wheel_y_offset} ${wheel_z_offset}" rpy="0 0 0"/>
   </xacro:wheel>
-  <!-- Front Right Wheel -->
-  <xacro:wheel prefix="front_right" parent="base_link">
+  <!-- Front Right Wheel - friction direction (1, 1, 0) -->
+  <xacro:wheel prefix="front_right" parent="base_link" friction_dir="1 1 0">
     <origin xyz="${wheel_x_offset_front} ${-wheel_y_offset} ${wheel_z_offset}" rpy="0 0 0"/>
   </xacro:wheel>
-  <!-- Rear Left Wheel -->
-  <xacro:wheel prefix="rear_left" parent="base_link">
+  <!-- Rear Left Wheel - friction direction (1, 1, 0) -->
+  <xacro:wheel prefix="rear_left" parent="base_link" friction_dir="1 1 0">
     <origin xyz="${wheel_x_offset_rear} ${wheel_y_offset} ${wheel_z_offset}" rpy="0 0 0"/>
   </xacro:wheel>
-  <!-- Rear Right Wheel -->
-  <xacro:wheel prefix="rear_right" parent="base_link">
+  <!-- Rear Right Wheel - friction direction (1, -1, 0) -->
+  <xacro:wheel prefix="rear_right" parent="base_link" friction_dir="1 -1 0">
     <origin xyz="${wheel_x_offset_rear} ${-wheel_y_offset} ${wheel_z_offset}" rpy="0 0 0"/>
   </xacro:wheel>
@@ -172,8 +177,12 @@
   <!-- Gazebo Plugins for gz sim (Gazebo Harmonic) -->
   <!-- ========================================== -->
-  <!-- Mecanum / Omni-Directional Drive controller plugin -->
+  <!-- ========================================== -->
+  <!-- Mecanum Drive Plugin                      -->
+  <!-- ========================================== -->
   <gazebo>
     <plugin filename="gz-sim-mecanum-drive-system" name="gz::sim::systems::MecanumDrive">
-      <!-- Wheel joint configuration (mecanum pattern) -->
+      <!-- Topic for velocity commands -->
+      <topic>cmd_vel</topic>
+      <!-- Wheel joint names (must match your URDF) -->
       <front_left_joint>wheel_front_left_joint</front_left_joint>
       <front_right_joint>wheel_front_right_joint</front_right_joint>
@@ -184,26 +193,33 @@
       <wheelbase>${wheelbase}</wheelbase>
       <wheel_radius>${wheel_radius}</wheel_radius>
-      <!-- Velocity limits -->
-      <max_linear_velocity>1.6</max_linear_velocity>
-      <min_linear_velocity>-1.6</min_linear_velocity>
-      <max_angular_velocity>4.5</max_angular_velocity>
-      <min_angular_velocity>-4.5</min_angular_velocity>
-      <!-- Acceleration limits -->
-      <max_linear_acceleration>1.5</max_linear_acceleration>
-      <max_angular_acceleration>3.0</max_angular_acceleration>
-      <!-- ROS 2 topics -->
-      <topic>cmd_vel</topic>
+      <!-- Control limits -->
+      <min_acceleration>-5</min_acceleration>
+      <max_acceleration>5</max_acceleration>
+      <!-- Odometry configuration -->
       <odom_topic>odom</odom_topic>
       <tf_topic>/tf</tf_topic>
-      <!-- Frame configuration -->
       <frame_id>odom</frame_id>
       <child_frame_id>base_footprint</child_frame_id>
-      <!-- Publishing configuration -->
       <odom_publish_frequency>50</odom_publish_frequency>
-      <publish_odom>true</publish_odom>
-      <publish_odom_tf>true</publish_odom_tf>
-    </plugin>
-  </gazebo>
-  <!-- Joint state publisher plugin -->
+    </plugin>
+  </gazebo>
+  <!-- ========================================== -->
+  <!-- Odometry Publisher Plugin                  -->
+  <!-- ========================================== -->
+  <gazebo>
+    <plugin name="gz::sim::systems::OdometryPublisher" filename="gz-sim-odometry-publisher-system">
+      <odom_topic>odom</odom_topic>
+      <odom_frame>odom</odom_frame>
+      <robot_base_frame>base_footprint</robot_base_frame>
+      <publish_tf>true</publish_tf>
+      <tf_topic>tf</tf_topic>
+      <odom_publish_frequency>50</odom_publish_frequency>
+      <xyz_offset>0 0 0</xyz_offset>
+      <rpy_offset>0 0 0</rpy_offset>
+    </plugin>
+  </gazebo>
+  <!-- ========================================== -->
+  <!-- Joint State Publisher Plugin               -->
+  <!-- ========================================== -->
   <gazebo>
     <plugin filename="gz-sim-joint-state-publisher-system" name="gz::sim::systems::JointStatePublisher">
@@ -216,5 +232,8 @@
     </plugin>
   </gazebo>
-  <!-- Pose publisher plugin -->
+  <!-- ========================================== -->
+  <!-- Pose Publisher Plugin (optional)           -->
+  <!-- Enable to publish robot pose information   -->
+  <!-- ========================================== -->
   <gazebo>
     <plugin filename="gz-sim-pose-publisher-system" name="gz::sim::systems::PosePublisher">

File: ros2_ws/src/avg_description/urdf/wheel_macro.xacro (robot description, xacro)
@@ -1,14 +1,14 @@
 <?xml version="1.0"?>
-<robot xmlns:xacro="http://www.ros.org/wiki/xacro">
+<robot xmlns:xacro="http://www.ros.org/wiki/xacro" xmlns:gz="http://gazebosim.org/schema">
   <!--
-    Wheel Macro
-    Creates a wheel with visual, collision, and inertial properties
+    Wheel Macro for Mecanum Drive
+    Creates a mecanum wheel with visual, collision, and inertial properties
     Parameters:
-      - prefix: wheel position identifier (e.g., front_left, rear_right)
+      - prefix: wheel position identifier (front_left, rear_left, front_right, rear_right)
       - parent: parent link name
-      - xyz: position offset [x, y, z]
-      - rpy: orientation [roll, pitch, yaw]
+      - origin: position and orientation block
+      - friction_dir: friction direction vector for mecanum physics
   -->
-  <xacro:macro name="wheel" params="prefix parent *origin">
+  <xacro:macro name="wheel" params="prefix parent friction_dir *origin">
     <!-- Wheel properties -->
     <xacro:property name="wheel_radius" value="0.05"/>
@@ -70,8 +70,9 @@
         <material name="dark_grey"/>
       </visual>
+      <!-- Collision with sphere for better mecanum simulation -->
       <collision>
-        <origin xyz="0 0 0" rpy="${pi/2} 0 0"/>
+        <origin xyz="0 0 0" rpy="0 0 0"/>
         <geometry>
-          <cylinder radius="${wheel_radius}" length="${wheel_width}"/>
+          <sphere radius="${wheel_radius}"/>
         </geometry>
       </collision>
@@ -96,24 +97,19 @@
       <dynamics damping="0.05" friction="0.05"/>
     </joint>
-    <!-- Gazebo properties for MECANUM/OMNI wheel physics -->
+    <!-- Gazebo properties for MECANUM wheel physics -->
     <gazebo reference="wheel_${prefix}">
       <material>Gazebo/Black</material>
-      <!-- Omnidirectional friction (equal in all directions for mecanum) -->
-      <mu1>1.0</mu1>   <!-- Primary friction -->
-      <mu2>1.0</mu2>   <!-- Secondary friction (equal for omni movement) -->
-      <!-- Contact physics - Optimized for mecanum -->
-      <kp>1000000.0</kp>     <!-- Contact stiffness -->
-      <kd>10.0</kd>          <!-- Contact damping -->
-      <minDepth>0.001</minDepth>
-      <maxVel>100.0</maxVel>
-      <maxContacts>1</maxContacts>  <!-- Single contact point per wheel -->
-      <!-- Mecanum wheels need some slip in all directions -->
-      <slip1>0.1</slip1>
-      <slip2>0.1</slip2>
-      <!-- Surface properties for consistent behavior -->
-      <bounce>0.0</bounce>
-      <bounce_threshold>100000</bounce_threshold>
-      <soft_cfm>0.0</soft_cfm>
-      <soft_erp>0.2</soft_erp>
+      <!-- Mecanum-specific friction with directional vector -->
+      <collision>
+        <surface>
+          <friction>
+            <ode>
+              <mu>1.5</mu>
+              <mu2>0.0</mu2>
+              <fdir1 gz:expressed_in="base_footprint">${friction_dir}</fdir1>
+            </ode>
+          </friction>
+        </surface>
+      </collision>
     </gazebo>
   </xacro:macro>
