Commit message: feat(amr_description): add dual drive modes and enhance documentation
- Implement dual drive system (Differential and Mecanum) in URDF
- Add `drive_mode` argument to `sim.launch.py` and `display.launch.py`
- Update `wheel_macro.xacro` to support anisotropic friction for mecanum wheels
- Configure `robot.xacro` to switch Gazebo plugins based on drive mode
- Overhaul README.md with professional visual gallery, badges, and diagrams
- Add documentation images for robot model, sensor views, and simulation worlds

File: ros2_ws/src/amr_description/urdf/robot.xacro (robot description, xacro)
@@ -1,4 +1,16 @@
 <?xml version="1.0"?>
-<robot name="warehouse_agv" xmlns:xacro="http://www.ros.org/wiki/xacro">
+<!--
+  Warehouse AMR Robot Description
+  This file defines the URDF/Xacro model for a warehouse autonomous mobile robot.
+  It supports two drive modes:
+  1. Differential Drive (default): Standard 4-wheel skid-steer configuration.
+  2. Mecanum Drive: Omnidirectional drive using mecanum wheels (useful for SLAM/Mapping).
+  Usage:
+    xacro robot.xacro drive_mode:=diff    (Differential Drive)
+    xacro robot.xacro drive_mode:=mecanum (Mecanum Drive)
+-->
+<robot name="warehouse_amr" xmlns:xacro="http://www.ros.org/wiki/xacro">
+  <!-- Arguments -->
+  <xacro:arg name="drive_mode" default="diff"/>
   <!-- Include all macro files -->
   <xacro:include filename="$(find amr_description)/urdf/materials.xacro"/>
@@ -19,4 +31,14 @@
   <xacro:property name="wheel_y_offset" value="${wheel_separation/2 + wheel_width/2}"/>
   <xacro:property name="wheel_z_offset" value="0"/>
+  <!-- Drive Mode Configuration -->
+  <xacro:property name="drive_mode" value="$(arg drive_mode)"/>
+  <xacro:if value="${drive_mode == 'mecanum'}">
+    <xacro:property name="wheel_mu1" value="1.5"/>
+    <xacro:property name="wheel_mu2" value="0.0"/>
+  </xacro:if>
+  <xacro:unless value="${drive_mode == 'mecanum'}">
+    <xacro:property name="wheel_mu1" value="1.0"/>
+    <xacro:property name="wheel_mu2" value="1.0"/>
+  </xacro:unless>
   <!-- ========================================== -->
   <!-- Base Footprint Link (ground projection)    -->
@@ -141,20 +163,20 @@
   </gazebo>
   <!-- ========================================== -->
-  <!-- Wheels (Using Wheel Macro with Mecanum Friction) -->
+  <!-- Wheels with Mecanum Friction               -->
   <!-- ========================================== -->
   <!-- Front Left Wheel - friction direction (1, -1, 0) -->
-  <xacro:wheel prefix="front_left" parent="base_link" friction_dir="1 -1 0">
+  <xacro:wheel prefix="front_left" parent="base_link" friction_dir="1 -1 0" mu1="${wheel_mu1}" mu2="${wheel_mu2}">
     <origin xyz="${wheel_x_offset_front} ${wheel_y_offset} ${wheel_z_offset}" rpy="0 0 0"/>
   </xacro:wheel>
   <!-- Front Right Wheel - friction direction (1, 1, 0) -->
-  <xacro:wheel prefix="front_right" parent="base_link" friction_dir="1 1 0">
+  <xacro:wheel prefix="front_right" parent="base_link" friction_dir="1 1 0" mu1="${wheel_mu1}" mu2="${wheel_mu2}">
     <origin xyz="${wheel_x_offset_front} ${-wheel_y_offset} ${wheel_z_offset}" rpy="0 0 0"/>
   </xacro:wheel>
   <!-- Rear Left Wheel - friction direction (1, 1, 0) -->
-  <xacro:wheel prefix="rear_left" parent="base_link" friction_dir="1 1 0">
+  <xacro:wheel prefix="rear_left" parent="base_link" friction_dir="1 1 0" mu1="${wheel_mu1}" mu2="${wheel_mu2}">
     <origin xyz="${wheel_x_offset_rear} ${wheel_y_offset} ${wheel_z_offset}" rpy="0 0 0"/>
   </xacro:wheel>
   <!-- Rear Right Wheel - friction direction (1, -1, 0) -->
-  <xacro:wheel prefix="rear_right" parent="base_link" friction_dir="1 -1 0">
+  <xacro:wheel prefix="rear_right" parent="base_link" friction_dir="1 -1 0" mu1="${wheel_mu1}" mu2="${wheel_mu2}">
     <origin xyz="${wheel_x_offset_rear} ${-wheel_y_offset} ${wheel_z_offset}" rpy="0 0 0"/>
   </xacro:wheel>
@@ -180,43 +202,72 @@
   <!-- Mecanum Drive Plugin                      -->
   <!-- ========================================== -->
-  <gazebo>
-    <plugin filename="gz-sim-mecanum-drive-system" name="gz::sim::systems::MecanumDrive">
-      <!-- Topic for velocity commands -->
-      <topic>cmd_vel</topic>
-      <!-- Wheel joint names (must match your URDF) -->
-      <front_left_joint>wheel_front_left_joint</front_left_joint>
-      <front_right_joint>wheel_front_right_joint</front_right_joint>
-      <back_left_joint>wheel_rear_left_joint</back_left_joint>
-      <back_right_joint>wheel_rear_right_joint</back_right_joint>
-      <!-- Robot physical parameters -->
-      <wheel_separation>${wheel_separation}</wheel_separation>
-      <wheelbase>${wheelbase}</wheelbase>
-      <wheel_radius>${wheel_radius}</wheel_radius>
-      <!-- Control limits -->
-      <min_acceleration>-5</min_acceleration>
-      <max_acceleration>5</max_acceleration>
-      <!-- Odometry configuration -->
-      <odom_topic>odom</odom_topic>
-      <tf_topic>/tf</tf_topic>
-      <frame_id>odom</frame_id>
-      <child_frame_id>base_footprint</child_frame_id>
-      <odom_publish_frequency>50</odom_publish_frequency>
-    </plugin>
-  </gazebo>
+  <xacro:if value="${drive_mode == 'mecanum'}">
+    <gazebo>
+      <plugin filename="gz-sim-mecanum-drive-system" name="gz::sim::systems::MecanumDrive">
+        <!-- Topic for velocity commands -->
+        <topic>cmd_vel</topic>
+        <!-- Wheel joint names (must match your URDF) -->
+        <front_left_joint>wheel_front_left_joint</front_left_joint>
+        <front_right_joint>wheel_front_right_joint</front_right_joint>
+        <back_left_joint>wheel_rear_left_joint</back_left_joint>
+        <back_right_joint>wheel_rear_right_joint</back_right_joint>
+        <!-- Robot physical parameters -->
+        <wheel_separation>${wheel_separation}</wheel_separation>
+        <wheelbase>${wheelbase}</wheelbase>
+        <wheel_radius>${wheel_radius}</wheel_radius>
+        <!-- Control limits -->
+        <min_acceleration>-5</min_acceleration>
+        <max_acceleration>5</max_acceleration>
+        <!-- Odometry configuration -->
+        <odom_topic>odom</odom_topic>
+        <tf_topic>/tf</tf_topic>
+        <frame_id>odom</frame_id>
+        <child_frame_id>base_footprint</child_frame_id>
+        <odom_publish_frequency>50</odom_publish_frequency>
+      </plugin>
+    </gazebo>
+  </xacro:if>
+  <!-- ========================================== -->
+  <!-- Differential Drive Plugin                  -->
+  <!-- ========================================== -->
+  <xacro:unless value="${drive_mode == 'mecanum'}">
+    <gazebo>
+      <plugin filename="gz-sim-diff-drive-system" name="gz::sim::systems::DiffDrive">
+        <!-- Topic for velocity commands -->
+        <topic>cmd_vel</topic>
+        <!-- Wheel joint names -->
+        <left_joint>wheel_front_left_joint</left_joint>
+        <left_joint>wheel_rear_left_joint</left_joint>
+        <right_joint>wheel_front_right_joint</right_joint>
+        <right_joint>wheel_rear_right_joint</right_joint>
+        <!-- Robot physical parameters -->
+        <wheel_separation>${wheel_separation}</wheel_separation>
+        <wheel_radius>${wheel_radius}</wheel_radius>
+        <!-- Odometry configuration -->
+        <odom_topic>odom</odom_topic>
+        <tf_topic>/tf</tf_topic>
+        <frame_id>odom</frame_id>
+        <child_frame_id>base_footprint</child_frame_id>
+        <odom_publish_frequency>50</odom_publish_frequency>
+      </plugin>
+    </gazebo>
+  </xacro:unless>
   <!-- ========================================== -->
   <!-- Odometry Publisher Plugin                  -->
   <!-- ========================================== -->
-  <gazebo>
-    <plugin name="gz::sim::systems::OdometryPublisher" filename="gz-sim-odometry-publisher-system">
-      <odom_topic>odom</odom_topic>
-      <odom_frame>odom</odom_frame>
-      <robot_base_frame>base_footprint</robot_base_frame>
-      <publish_tf>true</publish_tf>
-      <tf_topic>tf</tf_topic>
-      <odom_publish_frequency>50</odom_publish_frequency>
-      <xyz_offset>0 0 0</xyz_offset>
-      <rpy_offset>0 0 0</rpy_offset>
-    </plugin>
-  </gazebo>
+  <xacro:if value="${drive_mode == 'mecanum'}">
+    <gazebo>
+      <plugin name="gz::sim::systems::OdometryPublisher" filename="gz-sim-odometry-publisher-system">
+        <odom_topic>odom</odom_topic>
+        <odom_frame>odom</odom_frame>
+        <robot_base_frame>base_footprint</robot_base_frame>
+        <publish_tf>true</publish_tf>
+        <tf_topic>tf</tf_topic>
+        <odom_publish_frequency>50</odom_publish_frequency>
+        <xyz_offset>0 0 0</xyz_offset>
+        <rpy_offset>0 0 0</rpy_offset>
+      </plugin>
+    </gazebo>
+  </xacro:if>
   <!-- ========================================== -->
   <!-- Joint State Publisher Plugin               -->

File: ros2_ws/src/amr_description/urdf/wheel_macro.xacro (robot description, xacro)
@@ -2,13 +2,16 @@
 <robot xmlns:xacro="http://www.ros.org/wiki/xacro" xmlns:gz="http://gazebosim.org/schema">
   <!--
-    Wheel Macro for Mecanum Drive
-    Creates a mecanum wheel with visual, collision, and inertial properties
+    Wheel Macro
+    Creates a wheel with visual, collision, and inertial properties.
+    Supports both standard friction (for diff drive) and directional friction (for mecanum drive).
     Parameters:
       - prefix: wheel position identifier (front_left, rear_left, front_right, rear_right)
       - parent: parent link name
+      - friction_dir: friction direction vector for mecanum physics (e.g., "1 1 0")
+      - mu1: friction coefficient in fdir1 direction (default: 1.5)
+      - mu2: friction coefficient in perpendicular direction (default: 0.0)
       - origin: position and orientation block
-      - friction_dir: friction direction vector for mecanum physics
   -->
-  <xacro:macro name="wheel" params="prefix parent friction_dir *origin">
+  <xacro:macro name="wheel" params="prefix parent friction_dir mu1:=1.5 mu2:=0.0 *origin">
     <!-- Wheel properties -->
     <xacro:property name="wheel_radius" value="0.05"/>
@@ -97,14 +100,14 @@
       <dynamics damping="0.05" friction="0.05"/>
     </joint>
-    <!-- Gazebo properties for MECANUM wheel physics -->
+    <!-- Gazebo properties for wheel physics -->
     <gazebo reference="wheel_${prefix}">
       <material>Gazebo/Black</material>
-      <!-- Mecanum-specific friction with directional vector -->
+      <!-- Wheel friction properties -->
       <collision>
         <surface>
           <friction>
             <ode>
-              <mu>1.5</mu>
-              <mu2>0.0</mu2>
+              <mu>${mu1}</mu>
+              <mu2>${mu2}</mu2>
               <fdir1 gz:expressed_in="base_footprint">${friction_dir}</fdir1>
             </ode>
